File: atari_st.kicad_sch (KiCad schematic)
At the start: 2 parts, among them J5 ADAPTER, J6 ATARI

Commit message: a
Parts:
- J5: footprint Connector_IDC:IDC-Header_2x08_P2.54mm_Vertical -> Connector_IDC:IDC-Header_2x07_P2.54mm_Vertical; symbol Connector_Generic:Conn_01x16 -> Connector_Generic:Conn_01x14
Connections:
- net GND: no longer J5.16 (Pin_16)
- no-connect marks 3 -> 0
Changed lines of the file:
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@@
   (paper "A4")
   (junction (at 138.43 87.63) (diameter 0.9144) (color 0 0 0 0))
-  (no_connect (at 121.92 52.07))
-  (no_connect (at 121.92 85.09))
-  (no_connect (at 92.71 87.63))
   (wire (pts (xy 92.71 52.07) (xy 121.92 52.07))
     (stroke (width 0) (type solid) (color 0 0 0 0))
@@
   )
   (wire (pts (xy 92.71 82.55) (xy 135.89 82.55))
-    (stroke (width 0) (type solid) (color 0 0 0 0))
-  )
-  (wire (pts (xy 95.25 90.17) (xy 92.71 90.17))
-    (stroke (width 0) (type solid) (color 0 0 0 0))
-  )
-  (wire (pts (xy 95.25 95.25) (xy 95.25 90.17))
     (stroke (width 0) (type solid) (color 0 0 0 0))
   )
@@
     (effects (font (size 1.27 1.27)) (justify right bottom))
   )
-  (symbol (lib_id "power:GND") (at 95.25 95.25 0) (unit 1)
-    (in_bom yes) (on_board yes)
-    (property "Reference" "#PWR0103" (id 0) (at 95.25 101.6 0)
-      (effects (font (size 1.27 1.27)) hide)
-    )
-    (property "Value" "GND" (id 1) (at 96.52 100.33 0))
-    (property "Footprint" "" (id 2) (at 95.25 95.25 0)
-      (effects (font (size 1.27 1.27)) hide)
-    )
-    (property "Datasheet" "" (id 3) (at 95.25 95.25 0)
-      (effects (font (size 1.27 1.27)) hide)
-    )
-  )
   (symbol (lib_id "power:GND") (at 127 95.25 0) (unit 1)
     (in_bom yes) (on_board yes)
@@
     )
     (property "Datasheet" "" (id 3) (at 127 95.25 0)
+      (effects (font (size 1.27 1.27)) hide)
+    )
+  )
+  (symbol (lib_id "Connector_Generic:Conn_01x14") (at 87.63 67.31 0) (mirror y) (unit 1)
+    (in_bom yes) (on_board yes)
+    (property "Reference" "J5" (id 0) (at 90.17 43.18 0))
+    (property "Value" "ADAPTER" (id 1) (at 90.17 45.72 0))
+    (property "Footprint" "Connector_IDC:IDC-Header_2x07_P2.54mm_Vertical" (id 2) (at 87.63 67.31 0)
+      (effects (font (size 1.27 1.27)) hide)
+    )
+    (property "Datasheet" "~" (id 3) (at 87.63 67.31 0)
       (effects (font (size 1.27 1.27)) hide)
     )
@@
       (effects (font (size 1.27 1.27)) hide)
     )
-  )
-  (symbol (lib_id "Connector_Generic:Conn_01x16") (at 87.63 69.85 0) (mirror y) (unit 1)
-    (in_bom yes) (on_board yes)
-    (property "Reference" "J5" (id 0) (at 90.17 45.72 0))
-    (property "Value" "ADAPTER" (id 1) (at 90.17 48.26 0))
-    (property "Footprint" "Connector_IDC:IDC-Header_2x08_P2.54mm_Vertical" (id 2) (at 87.63 69.85 0)
-      (effects (font (size 1.27 1.27)) hide)
-    )
-    (property "Datasheet" "~" (id 3) (at 87.63 69.85 0)
-      (effects (font (size 1.27 1.27)) hide)
-    )
