File: floppy.kicad_sch (KiCad schematic)
At the start: 13 parts, among them J1 12VDC, J2 FLOPPY_PWR, J3 ADAPTER, J4 FLOPPY, SW1 SW_DPDT_x2, U1 L7805

Commit message: a
Parts:
- J3: footprint Connector_IDC:IDC-Header_2x08_P2.54mm_Horizontal -> Connector_IDC:IDC-Header_2x07_P2.54mm_Horizontal; symbol Connector_Generic:Conn_01x16 -> Connector_Generic:Conn_01x14
Connections:
- net GND: no longer J3.16 (Pin_16)
- no-connect marks 5 -> 4
Changed lines of the file:
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@@
   (no_connect (at 121.92 59.69))
   (no_connect (at 134.62 44.45))
-  (no_connect (at 92.71 87.63))
   (wire (pts (xy 26.67 63.5) (xy 26.67 60.96))
     (stroke (width 0) (type solid) (color 0 0 0 0))
@@
   )
   (wire (pts (xy 92.71 80.01) (xy 121.92 80.01))
-    (stroke (width 0) (type solid) (color 0 0 0 0))
-  )
-  (wire (pts (xy 92.71 90.17) (xy 95.25 90.17))
     (stroke (width 0) (type solid) (color 0 0 0 0))
   )
@@
     )
     (property "Datasheet" "" (id 3) (at 62.23 43.18 0)
-      (effects (font (size 1.27 1.27)) hide)
-    )
-  )
-  (symbol (lib_id "power:GND") (at 95.25 90.17 0) (unit 1)
-    (in_bom yes) (on_board yes)
-    (property "Reference" "#PWR0102" (id 0) (at 95.25 96.52 0)
-      (effects (font (size 1.27 1.27)) hide)
-    )
-    (property "Value" "GND" (id 1) (at 96.52 95.25 0))
-    (property "Footprint" "" (id 2) (at 95.25 90.17 0)
-      (effects (font (size 1.27 1.27)) hide)
-    )
-    (property "Datasheet" "" (id 3) (at 95.25 90.17 0)
       (effects (font (size 1.27 1.27)) hide)
     )
@@
     )
   )
-  (symbol (lib_id "Connector_Generic:Conn_01x16") (at 87.63 69.85 0) (mirror y) (unit 1)
-    (in_bom yes) (on_board yes)
-    (property "Reference" "J3" (id 0) (at 90.17 45.72 0))
-    (property "Value" "ADAPTER" (id 1) (at 90.17 48.26 0))
-    (property "Footprint" "Connector_IDC:IDC-Header_2x08_P2.54mm_Horizontal" (id 2) (at 87.63 69.85 0)
-      (effects (font (size 1.27 1.27)) hide)
-    )
-    (property "Datasheet" "~" (id 3) (at 87.63 69.85 0)
+  (symbol (lib_id "Connector_Generic:Conn_01x14") (at 87.63 67.31 0) (mirror y) (unit 1)
+    (in_bom yes) (on_board yes)
+    (property "Reference" "J3" (id 0) (at 90.17 43.18 0))
+    (property "Value" "ADAPTER" (id 1) (at 90.17 45.72 0))
+    (property "Footprint" "Connector_IDC:IDC-Header_2x07_P2.54mm_Horizontal" (id 2) (at 87.63 67.31 0)
+      (effects (font (size 1.27 1.27)) hide)
+    )
+    (property "Datasheet" "~" (id 3) (at 87.63 67.31 0)
       (effects (font (size 1.27 1.27)) hide)
     )
@@
       (reference "#PWR07") (unit 1) (value "GND") (footprint "")
     )
-    (path "/ceeac992-fc29-4a73-9f03-f51f466531c4"
-      (reference "#PWR0102") (unit 1) (value "GND") (footprint "")
-    )
     (path "/86c8debe-a504-4f15-b922-97104be1137e"
       (reference "#PWR0104") (unit 1) (value "GND") (footprint "")
@@
     )
     (path "/afba136e-7f84-4ff1-b6f4-6a1445c64da2"
-      (reference "J3") (unit 1) (value "ADAPTER") (footprint "Connector_IDC:IDC-Header_2x08_P2.54mm_Horizontal")
+      (reference "J3") (unit 1) (value "ADAPTER") (footprint "Connector_IDC:IDC-Header_2x07_P2.54mm_Horizontal")
     )
     (path "/00000000-0000-0000-0000-00005fc468f3"
@@
       (reference "#PWR0101") (unit 1) (value "GND") (footprint "")
     )
-    (path "/214e5bd1-de3c-4ec2-8553-5b0be1a71a0f/507d2933-082b-4fad-ad51-d42819335b4a"
-      (reference "#PWR0103") (unit 1) (value "GND") (footprint "")
-    )
     (path "/214e5bd1-de3c-4ec2-8553-5b0be1a71a0f/e4d3af14-b01c-4ff2-907e-cbfc6e32f0ec"
-      (reference "J5") (unit 1) (value "ADAPTER") (footprint "Connector_IDC:IDC-Header_2x08_P2.54mm_Vertical")
+      (reference "J5") (unit 1) (value "ADAPTER") (footprint "Connector_IDC:IDC-Header_2x07_P2.54mm_Vertical")
     )
     (path "/214e5bd1-de3c-4ec2-8553-5b0be1a71a0f/3e20fa31-0809-47c3-be37-022bd242ab1a"
