File: floppy.kicad_pcb (KiCad board)
At the start: 2 copper layers, 96.5 x 44.5 mm, 13 parts, among them J1 12VDC, J2 FLOPPY_PWR, J3 ADAPTER, J4 FLOPPY, SW1 SW_DPDT_x2, U1 L7805

Commit message: a
Parts:
- added J5: ADAPTER, Connector_IDC:IDC-Header_2x07_P2.54mm_Vertical, F.Cu at (166.2, 77.8)
- added J6: ATARI, parts:DIN14, F.Cu at (158.6, 89.0)
- C1: footprint Capacitor_THT:CP_Radial_D10.0mm_P5.00mm -> Capacitor_THT:C_Radial_D10.0mm_H12.5mm_P5.00mm
- J2: footprint Connector_PinHeader_2.54mm:PinHeader_1x04_P2.54mm_Vertical -> Connector_Molex:Molex_KK-254_AE-6410-04A_1x04_P2.54mm_Vertical
- J3: footprint Connector_IDC:IDC-Header_2x08_P2.54mm_Horizontal -> Connector_IDC:IDC-Header_2x07_P2.54mm_Horizontal
- turned J2 to 0 degrees
Connections:
- net no_connect_36 renamed no_connect_(J4-Pad1)
- net no_connect_37 renamed no_connect_(J4-Pad14)
- net no_connect_38 renamed no_connect_(J4-Pad4)
- net no_connect_39 renamed no_connect_(J4-Pad6)

Commit message: there was shrinkage
Parts:
- moved H2 5.59 mm to (41.2, 104.1)
- moved H4 5.59 mm to (41.2, 67.3)
- moved U1 4.62 mm to (52.2, 87.0)
- moved C2 1.96 mm to (57.2, 92.8)
- moved J1 1.96 mm to (57.2, 76.8)
- moved J2 1.96 mm to (57.2, 99.1)
- moved C1 1.95 mm to (65.3, 92.8)
- moved D1 1.95 mm to (49.6, 81.9)
- moved H1 1.11 mm to (123.3, 67.3)
- moved H3 1.11 mm to (123.3, 104.1)
Routing:
- net +5V: track 22.6 -> 20.1 mm
- net +12V: track 29.8 -> 28.2 mm
Other:
- board size 96.5 x 44.5 mm -> 89.8 x 44.5 mm
Changed lines of the file:
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@@
   )
   (footprint "Package_TO_SOT_THT:TO-220-3_Horizontal_TabDown" (layer "F.Cu")
-    (at 47.625 86.995 180)
+    (at 52.25 86.995 180)
     (descr "TO-220-3, Horizontal, RM 2.54mm, see https://www.vishay.com/docs/66542/to-220-1.pdf")
     (tags "TO-220-3 Horizontal RM 2.54mm")
@@
   )
   (footprint "Diode_THT:D_DO-41_SOD81_P7.62mm_Horizontal" (layer "F.Cu")
-    (at 47.625 81.915)
+    (at 49.58 81.915)
     (descr "Diode, DO-41_SOD81 series, Axial, Horizontal, pin pitch=7.62mm, , length*diameter=5.2*2.7mm^2, , http://www.diodes.com/_files/packages/DO-41%20(Plastic).pdf")
     (tags "Diode DO-41_SOD81 series Axial Horizontal pin pitch 7.62mm  length 5.2mm diameter 2.7mm")
@@
   )
   (footprint "Connector_Molex:Molex_KK-254_AE-6410-04A_1x04_P2.54mm_Vertical" (layer "F.Cu")
-    (at 55.245 99.1)
+    (at 57.2 99.1)
     (descr "Molex KK-254 Interconnect System, old/engineering part number: AE-6410-04A example for new part number: 22-27-2041, 4 Pins (http://www.molex.com/pdm_docs/sd/022272021_sd.pdf), generated with kicad-footprint-generator")
     (tags "connector Molex KK-254 vertical")
@@
   )
   (footprint "Connector_BarrelJack:BarrelJack_Horizontal" (layer "F.Cu")
-    (at 55.245 76.835 -90)
+    (at 57.2 76.835 -90)
     (descr "DC Barrel Jack")
     (tags "Power Jack")
@@
   )
   (footprint "MountingHole:MountingHole_3.2mm_M3_DIN965_Pad_TopBottom" (layer "F.Cu")
-    (at 124.46 67.31)
+    (at 123.345 67.31)
     (descr "Mounting Hole 3.2mm, M3, DIN965")
     (tags "mounting hole 3.2mm m3 din965")
@@
   )
   (footprint "Capacitor_THT:C_Disc_D10.0mm_W2.5mm_P5.00mm" (layer "F.Cu")
-    (at 55.245 92.75 90)
+    (at 57.2 92.75 90)
     (descr "C, Disc series, Radial, pin pitch=5.00mm, , diameter*width=10*2.5mm^2, Capacitor, http://cdn-reichelt.de/documents/datenblatt/B300/DS_KERKO_TC.pdf")
     (tags "C Disc series Radial pin pitch 5.00mm  diameter 10mm width 2.5mm Capacitor")
@@
   )
   (footprint "MountingHole:MountingHole_3.2mm_M3_DIN965_Pad_TopBottom" (layer "F.Cu")
-    (at 35.56 104.14)
+    (at 41.155 104.14)
     (descr "Mounting Hole 3.2mm, M3, DIN965")
     (tags "mounting hole 3.2mm m3 din965")
@@
   )
   (footprint "MountingHole:MountingHole_3.2mm_M3_DIN965_Pad_TopBottom" (layer "F.Cu")
-    (at 35.56 67.31)
+    (at 41.155 67.31)
     (descr "Mounting Hole 3.2mm, M3, DIN965")
     (tags "mounting hole 3.2mm m3 din965")
@@
   )
   (footprint "MountingHole:MountingHole_3.2mm_M3_DIN965_Pad_TopBottom" (layer "F.Cu")
-    (at 124.46 104.14)
+    (at 123.345 104.14)
     (descr "Mounting Hole 3.2mm, M3, DIN965")
     (tags "mounting hole 3.2mm m3 din965")
@@
   )
   (footprint "Capacitor_THT:C_Radial_D10.0mm_H12.5mm_P5.00mm" (layer "F.Cu")
-    (at 63.39 92.75 90)
+    (at 65.345 92.75 90)
     (descr "C, Radial series, Radial, pin pitch=5.00mm, diameter=10mm, height=12.5mm, Non-Polar Electrolytic Capacitor")
     (tags "C Radial series Radial pin pitch 5.00mm diameter 10mm height 12.5mm Non-Polar Electrolytic Capacitor")
@@
     )
   )
-  (gr_line (start 31.75 106.68) (end 31.75 64.77) (layer "Edge.Cuts") (width 0.1))
-  (gr_line (start 127 107.95) (end 33.02 107.95) (layer "Edge.Cuts") (width 0.1))
-  (gr_arc (start 62.12 104.18) (end 62.12 105.45) (angle -180) (layer "Edge.Cuts") (width 0.1))
-  (gr_line (start 33.02 63.5) (end 127 63.5) (layer "Edge.Cuts") (width 0.1))
-  (gr_line (start 128.27 64.77) (end 128.27 106.68) (layer "Edge.Cuts") (width 0.1))
-  (gr_line (start 31.75 64.77) (end 33.02 63.5) (layer "Edge.Cuts") (width 0.1))
-  (gr_line (start 127 107.95) (end 128.27 106.68) (layer "Edge.Cuts") (width 0.1))
-  (gr_line (start 62.12 105.45) (end 55.77 105.45) (layer "Edge.Cuts") (width 0.1))
-  (gr_arc (start 55.77 104.18) (end 55.77 102.91) (angle -180) (layer "Edge.Cuts") (width 0.1))
-  (gr_line (start 55.77 102.91) (end 62.12 102.91) (layer "Edge.Cuts") (width 0.1))
-  (gr_line (start 33.02 107.95) (end 31.75 106.68) (layer "Edge.Cuts") (width 0.1))
-  (gr_line (start 128.27 64.77) (end 127 63.5) (layer "Edge.Cuts") (width 0.1))
+  (gr_line (start 37.345 106.68) (end 37.345 64.77) (layer "Edge.Cuts") (width 0.1))
+  (gr_line (start 125.885 107.95) (end 38.615 107.95) (layer "Edge.Cuts") (width 0.1))
+  (gr_arc (start 64.075 104.18) (end 64.075 105.45) (angle -180) (layer "Edge.Cuts") (width 0.1))
+  (gr_line (start 38.615 63.5) (end 125.885 63.5) (layer "Edge.Cuts") (width 0.1))
+  (gr_line (start 127.155 64.77) (end 127.155 106.68) (layer "Edge.Cuts") (width 0.1))
+  (gr_line (start 37.345 64.77) (end 38.615 63.5) (layer "Edge.Cuts") (width 0.1))
+  (gr_line (start 125.885 107.95) (end 127.155 106.68) (layer "Edge.Cuts") (width 0.1))
+  (gr_line (start 64.075 105.45) (end 57.725 105.45) (layer "Edge.Cuts") (width 0.1))
+  (gr_arc (start 57.725 104.18) (end 57.725 102.91) (angle -180) (layer "Edge.Cuts") (width 0.1))
+  (gr_line (start 57.725 102.91) (end 64.075 102.91) (layer "Edge.Cuts") (width 0.1))
+  (gr_line (start 38.615 107.95) (end 37.345 106.68) (layer "Edge.Cuts") (width 0.1))
+  (gr_line (start 127.155 64.77) (end 125.885 63.5) (layer "Edge.Cuts") (width 0.1))
   (gr_text "REVERSED" (at 111 73.25 90) (layer "F.SilkS")
     (effects (font (size 1 1) (thickness 0.15)))
   )
-  (gr_text "GND" (at 58.695 106.75) (layer "F.SilkS")
+  (gr_text "GND" (at 60.65 106.75) (layer "F.SilkS")
     (effects (font (size 1 1) (thickness 0.2)))
   )
-  (gr_text "+12V" (at 63.14 106.75) (layer "F.SilkS")
+  (gr_text "+12V" (at 65.095 106.75) (layer "F.SilkS")
     (effects (font (size 1 1) (thickness 0.2)))
   )
@@
     (effects (font (size 1 1) (thickness 0.15)))
   )
-  (gr_text "+5V" (at 54.25 106.75) (layer "F.SilkS")
+  (gr_text "+5V" (at 56.205 106.75) (layer "F.SilkS")
     (effects (font (size 1 1) (thickness 0.2)))
   )
-  (segment (start 62.865 93.275) (end 62.865 99.1) (width 0.4) (layer "F.Cu") (net 2))
-  (segment (start 63.39 92.75) (end 62.865 93.275) (width 0.4) (layer "F.Cu") (net 2))
-  (segment (start 47.625 86.995) (end 47.625 81.915) (width 0.4) (layer "F.Cu") (net 2))
-  (segment (start 60.85 90.21) (end 50.84 90.21) (width 0.4) (layer "F.Cu") (net 2))
-  (segment (start 50.84 90.21) (end 47.625 86.995) (width 0.4) (layer "F.Cu") (net 2))
-  (segment (start 63.39 92.75) (end 60.85 90.21) (width 0.4) (layer "F.Cu") (net 2))
-  (segment (start 46.32 92.75) (end 55.245 92.75) (width 0.4) (layer "F.Cu") (net 3))
-  (segment (start 42.545 86.995) (end 42.545 88.975) (width 0.4) (layer "F.Cu") (net 3))
-  (segment (start 55.245 92.75) (end 55.245 99.1) (width 0.4) (layer "F.Cu") (net 3))
-  (segment (start 42.545 88.975) (end 46.32 92.75) (width 0.4) (layer "F.Cu") (net 3))
-  (segment (start 55.245 76.835) (end 55.245 81.915) (width 0.4) (layer "F.Cu") (net 4))
+  (segment (start 64.82 93.275) (end 64.82 99.1) (width 0.4) (layer "F.Cu") (net 2))
+  (segment (start 52.25 86.995) (end 55.465 90.21) (width 0.4) (layer "F.Cu") (net 2))
+  (segment (start 65.345 92.75) (end 64.82 93.275) (width 0.4) (layer "F.Cu") (net 2))
+  (segment (start 49.58 81.915) (end 49.58 84.325) (width 0.4) (layer "F.Cu") (net 2))
+  (segment (start 49.58 84.325) (end 52.25 86.995) (width 0.4) (layer "F.Cu") (net 2))
+  (segment (start 55.465 90.21) (end 62.805 90.21) (width 0.4) (layer "F.Cu") (net 2))
+  (segment (start 65.345 92.75) (end 62.805 90.21) (width 0.4) (layer "F.Cu") (net 2))
+  (segment (start 47.17 89.3325) (end 50.5875 92.75) (width 0.4) (layer "F.Cu") (net 3))
+  (segment (start 50.5875 92.75) (end 57.2 92.75) (width 0.4) (layer "F.Cu") (net 3))
+  (segment (start 47.17 86.995) (end 47.17 89.3325) (width 0.4) (layer "F.Cu") (net 3))
+  (segment (start 57.2 92.75) (end 57.2 99.1) (width 0.4) (layer "F.Cu") (net 3))
+  (segment (start 57.2 76.835) (end 57.2 81.915) (width 0.4) (layer "F.Cu") (net 4))
   (segment (start 96.52 73.02) (end 96.52 73.66) (width 0.4) (layer "F.Cu") (net 5))
   (segment (start 96.52 73.27) (end 89.099901 65.849901) (width 0.4) (layer "F.Cu") (net 5))
