File: atari/atari.kicad_pcb (KiCad board)
At the start: 2 copper layers, 2 parts, among them J5 ADAPTER, J6 ATARI

Commit message: a
Connections:
- J5 pad 1: /FLOPPY_DISKCHANGE -> /FLOPPY_READ_DATA
- J5 pad 10: /FLOPPY_TRACK_00 -> /FLOPPY_STEP
- J5 pad 11: /FLOPPY_WRITE_PROTECT -> /FLOPPY_WRITE_DATA
- J5 pad 12: /FLOPPY_READ_DATA -> /FLOPPY_WRITE_GATE
- J5 pad 13: /FLOPPY_SIDE_SELECT -> /FLOPPY_TRACK_00
- J5 pad 14: /FLOPPY_READY -> /FLOPPY_WRITE_PROTECT
- J5 pad 2: /FLOPPY_INDEX -> /FLOPPY_SIDE_SELECT
- J5 pad 3: /FLOPPY_SELECT_A -> /GND
- J5 pad 4: /FLOPPY_SELECT_B -> /FLOPPY_INDEX
- J5 pad 5: /FLOPPY_MOTOR_ON -> /FLOPPY_SELECT_A
- J5 pad 6: /FLOPPY_STEP_DIRECTION -> /FLOPPY_SELECT_B
- J5 pad 7: /FLOPPY_STEP -> /GND
- J5 pad 8: /FLOPPY_WRITE_DATA -> /FLOPPY_MOTOR_ON
- J5 pad 9: /FLOPPY_WRITE_GATE -> /FLOPPY_STEP_DIRECTION
- J6 pad 3: GND -> /GND
- J6 pad 7: GND -> /GND
Routing:
- net /GND: track 0.00 -> 30.4 mm
- net /FLOPPY_SIDE_SELECT: track 0.00 -> 28.0 mm
- net /FLOPPY_READ_DATA: track 0.00 -> 27.5 mm
- net /FLOPPY_INDEX: track 0.00 -> 22.9 mm
- net /FLOPPY_SELECT_B: track 0.00 -> 22.6 mm
- net /FLOPPY_SELECT_A: track 0.00 -> 21.3 mm
- net /FLOPPY_TRACK_00: track 0.00 -> 18.0 mm
- net /FLOPPY_MOTOR_ON: track 0.00 -> 17.8 mm
- net /FLOPPY_WRITE_PROTECT: track 0.00 -> 16.4 mm
- net /FLOPPY_STEP_DIRECTION: track 0.00 -> 16.4 mm
- net /FLOPPY_WRITE_DATA: track 0.00 -> 14.1 mm
- net /FLOPPY_WRITE_GATE: track 0.00 -> 12.6 mm
- net /FLOPPY_STEP: track 0.00 -> 8.30 mm
Other:
- board outline added: 26.7 x 26 mm
