File: floppy/floppy.kicad_pcb (KiCad board)
At the start: 2 copper layers, 89.8 x 44.5 mm, 15 parts, among them J1 12VDC, J2 FLOPPY_PWR, J3 ADAPTER, J4 FLOPPY, J5 ADAPTER, J6 ATARI, SW1 SW_DPDT_x2, U1 L7805

Commit message: break up boards
Parts:
- removed J5: ADAPTER, Connector_IDC:IDC-Header_2x07_P2.54mm_Vertical
- removed J6: ATARI, parts:DIN14
Connections:
- J1 pad 3: GND -> (no net)
- J4 pad 1: no_connect_(J4-Pad1) -> unconnected-(J4-Pad1)
- J4 pad 14: no_connect_(J4-Pad14) -> unconnected-(J4-Pad14)
- J4 pad 4: no_connect_(J4-Pad4) -> unconnected-(J4-Pad4)
- J4 pad 6: no_connect_(J4-Pad6) -> unconnected-(J4-Pad6)

Commit message: a
Connections:
- J3 pad 1: /FLOPPY_DISKCHANGE -> GND
- J4 pad 2: /FLOPPY_DISKCHANGE -> unconnected-(J4-Pad2)
Routing:
- net /FLOPPY_DISKCHANGE: track 49.7 -> 0.00 mm
Changed lines of the file:
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@@
   (net 16 "/FLOPPY_MOTOR_ON")
   (net 17 "/FLOPPY_SELECT_A")
-  (net 18 "/FLOPPY_DISKCHANGE")
+  (net 18 "unconnected-(J4-Pad2)")
   (net 19 "/F_INSEL_B")
   (net 20 "/F_INSEL_A")
@@
     (fp_line (start 4.38 4.76) (end -0.32 4.76) (layer "F.Fab") (width 0.1))
     (pad "1" thru_hole roundrect (at 0 0 90) (locked) (size 1.7 1.7) (drill 1) (layers *.Cu *.Mask) (roundrect_rratio 0.147059)
-      (net 18 "/FLOPPY_DISKCHANGE") (pinfunction "Pin_1") (pintype "passive"))
+      (net 1 "GND") (pinfunction "Pin_1") (pintype "passive"))
     (pad "2" thru_hole circle (at 2.54 0 90) (locked) (size 1.7 1.7) (drill 1) (layers *.Cu *.Mask)
       (net 11 "/FLOPPY_INDEX") (pinfunction "Pin_2") (pintype "passive"))
@@
       (net 21 "unconnected-(J4-Pad1)") (pinfunction "Pin_1") (pintype "passive+no_connect"))
     (pad "2" thru_hole circle (at 2.54 0 270) (locked) (size 1.7 1.7) (drill 1) (layers *.Cu *.Mask)
-      (net 18 "/FLOPPY_DISKCHANGE") (pinfunction "Pin_2") (pintype "passive"))
+      (net 18 "unconnected-(J4-Pad2)") (pinfunction "Pin_2") (pintype "passive"))
     (pad "3" thru_hole circle (at 0 2.54 270) (locked) (size 1.7 1.7) (drill 1) (layers *.Cu *.Mask)
       (net 1 "GND") (pinfunction "Pin_3") (pintype "passive"))
@@
   (segment (start 110.399991 70.350009) (end 112.25 68.5) (width 0.4) (layer "B.Cu") (net 17))
   (segment (start 87.819988 70.35001) (end 110.399991 70.350009) (width 0.4) (layer "B.Cu") (net 17))
-  (segment (start 113.049999 105.390001) (end 103.539999 105.390001) (width 0.4) (layer "B.Cu") (net 18))
-  (segment (start 114.3 104.14) (end 113.049999 105.390001) (width 0.4) (layer "B.Cu") (net 18))
-  (segment (start 103.539999 105.390001) (end 102.850001 104.700003) (width 0.4) (layer "B.Cu") (net 18))
-  (segment (start 102.850001 100.460001) (end 81.28 78.89) (width 0.4) (layer "B.Cu") (net 18))
-  (segment (start 81.28 78.89) (end 81.28 76.2) (width 0.4) (layer "B.Cu") (net 18))
-  (segment (start 102.850001 104.700003) (end 102.850001 100.460001) (width 0.4) (layer "B.Cu") (net 18))
   (segment (start 109.75 73.651458) (end 109.75 68.3) (width 0.4) (layer "F.Cu") (net 19))
   (segment (start 101.6 104.14) (end 102.850001 102.889999) (width 0.4) (layer "F.Cu") (net 19))
