File: floppy/floppy.kicad_sch (KiCad schematic)
At the start: 13 parts, among them J1 12VDC, J2 FLOPPY_PWR, J3 ADAPTER, J4 FLOPPY, SW1 SW_DPDT_x2, U1 L7805

Commit message: break up boards
Other:
- removed sheet Atari ST
Changed lines of the file:
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@@
-(kicad_sch (version 20201015) (generator eeschema)
+(kicad_sch (version 20210126) (generator eeschema)
   (paper "A4")
   (junction (at 30.48 63.5) (diameter 0.9144) (color 0 0 0 0))
@@
       (effects (font (size 1.27 1.27)) hide)
     )
+    (pin "1")
   )
   (symbol (lib_id "power:+12V") (at 34.29 60.96 0) (unit 1)
@@
       (effects (font (size 1.27 1.27)) hide)
     )
+    (pin "1")
   )
   (symbol (lib_id "power:+12V") (at 50.8 27.94 0) (unit 1)
@@
       (effects (font (size 1.27 1.27)) hide)
     )
+    (pin "1")
   )
   (symbol (lib_id "power:+5V") (at 73.66 27.94 0) (unit 1)
@@
       (effects (font (size 1.27 1.27)) hide)
     )
+    (pin "1")
   )
   (symbol (lib_id "power:GND") (at 30.48 71.12 0) (unit 1)
@@
       (effects (font (size 1.27 1.27)) hide)
     )
+    (pin "1")
   )
   (symbol (lib_id "power:GND") (at 62.23 43.18 0) (unit 1)
@@
       (effects (font (size 1.27 1.27)) hide)
     )
+    (pin "1")
   )
   (symbol (lib_id "power:GND") (at 113.03 133.35 0) (unit 1)
@@
       (effects (font (size 1.27 1.27)) hide)
     )
+    (pin "1")
   )
   (symbol (lib_id "power:GND") (at 134.62 90.17 0) (unit 1)
@@
       (effects (font (size 1.27 1.27)) hide)
     )
+    (pin "1")
   )
   (symbol (lib_id "Mechanical:MountingHole_Pad") (at 105.41 130.81 0) (unit 1)
@@
       (effects (font (size 1.27 1.27)) hide)
     )
+    (pin "1")
   )
   (symbol (lib_id "Mechanical:MountingHole_Pad") (at 110.49 130.81 0) (unit 1)
@@
       (effects (font (size 1.27 1.27)) hide)
     )
+    (pin "1")
   )
   (symbol (lib_id "Mechanical:MountingHole_Pad") (at 115.57 130.81 0) (unit 1)
@@
       (effects (font (size 1.27 1.27)) hide)
     )
+    (pin "1")
   )
   (symbol (lib_id "Mechanical:MountingHole_Pad") (at 120.65 130.81 0) (unit 1)
@@
       (effects (font (size 1.27 1.27)) hide)
     )
+    (pin "1")
   )
   (symbol (lib_id "Device:D") (at 43.18 31.75 180) (unit 1)
@@
       (effects (font (size 1.27 1.27)) hide)
     )
+    (pin "1")
+    (pin "2")
   )
   (symbol (lib_id "Device:C_Polarized") (at 50.8 35.56 0) (unit 1)
@@
       (effects (font (size 1.27 1.27)) hide)
     )
+    (pin "1")
+    (pin "2")
   )
   (symbol (lib_id "Device:C") (at 73.66 35.56 0) (unit 1)
@@
       (effects (font (size 1.27 1.27)) hide)
     )
+    (pin "1")
+    (pin "2")
   )
   (symbol (lib_id "Connector:Conn_01x04_Male") (at 29.21 68.58 90) (unit 1)
@@
       (effects (font (size 1.27 1.27)) hide)
     )
+    (pin "1")
+    (pin "2")
+    (pin "3")
+    (pin "4")
   )
   (symbol (lib_id "Switch:SW_DPDT_x2") (at 41.91 113.03 0) (mirror y) (unit 1)
@@
       (effects (font (size 1.27 1.27)) hide)
     )
+    (pin "1")
+    (pin "2")
+    (pin "3")
   )
   (symbol (lib_id "Switch:SW_DPDT_x2") (at 41.91 127 0) (mirror y) (unit 2)
@@
       (effects (font (size 1.27 1.27)) hide)
     )
+    (pin "4")
+    (pin "5")
+    (pin "6")
   )
   (symbol (lib_id "Connector:Jack-DC") (at 27.94 34.29 0) (unit 1)
@@
       (effects (font (size 1.27 1.27)) hide)
     )
+    (pin "1")
+    (pin "2")
   )
   (symbol (lib_id "Regulator_Linear:L7812") (at 62.23 31.75 0) (unit 1)
@@
       (effects (font (size 1.27 1.27)) hide)
     )
+    (pin "1")
+    (pin "2")
+    (pin "3")
   )
   (symbol (lib_id "Connector_Generic:Conn_01x14") (at 87.63 67.31 0) (mirror y) (unit 1)
@@
       (effects (font (size 1.27 1.27)) hide)
     )
+    (pin "1")
+    (pin "10")
+    (pin "11")
+    (pin "12")
+    (pin "13")
+    (pin "14")
+    (pin "2")
+    (pin "3")
+    (pin "4")
+    (pin "5")
+    (pin "6")
+    (pin "7")
+    (pin "8")
+    (pin "9")
   )
   (symbol (lib_id "Connector_Generic:Conn_02x17_Odd_Even") (at 129.54 64.77 0) (mirror y) (unit 1)
@@
       (effects (font (size 1.27 1.27)) hide)
     )
-  )
-  (sheet (at 189.23 48.26) (size 35.56 33.02)
-    (stroke (width 0.001) (type solid) (color 132 0 132 1))
-    (fill (color 255 255 255 0.0000))
-    (property "Sheet name" "Atari ST" (id 0) (at 189.23 47.6241 0)
-      (effects (font (size 1.27 1.27)) (justify left bottom))
-    )
-    (property "Sheet file" "atari_st.kicad_sch" (id 1) (at 189.23 81.7889 0)
-      (effects (font (size 1.27 1.27)) (justify left top))
-    )
+    (pin "1")
+    (pin "10")
+    (pin "11")
+    (pin "12")
+    (pin "13")
+    (pin "14")
+    (pin "15")
+    (pin "16")
+    (pin "17")
+    (pin "18")
+    (pin "19")
+    (pin "2")
+    (pin "20")
+    (pin "21")
+    (pin "22")
+    (pin "23")
+    (pin "24")
+    (pin "25")
+    (pin "26")
+    (pin "27")
+    (pin "28")
+    (pin "29")
+    (pin "3")
+    (pin "30")
+    (pin "31")
+    (pin "32")
+    (pin "33")
+    (pin "34")
+    (pin "4")
+    (pin "5")
+    (pin "6")
+    (pin "7")
+    (pin "8")
+    (pin "9")
   )
   (sheet_instances
     (path "/" (page "1"))
-    (path "/214e5bd1-de3c-4ec2-8553-5b0be1a71a0f/" (page "2"))
   )
   (symbol_instances
@@
       (reference "U1") (unit 1) (value "L7805") (footprint "Package_TO_SOT_THT:TO-220-3_Horizontal_TabDown")
     )
-    (path "/214e5bd1-de3c-4ec2-8553-5b0be1a71a0f/278b2b95-eb2b-4c5f-bd49-6d46efcc2c1d"
-      (reference "#PWR0101") (unit 1) (value "GND") (footprint "")
-    )
-    (path "/214e5bd1-de3c-4ec2-8553-5b0be1a71a0f/e4d3af14-b01c-4ff2-907e-cbfc6e32f0ec"
-      (reference "J5") (unit 1) (value "ADAPTER") (footprint "Connector_IDC:IDC-Header_2x07_P2.54mm_Vertical")
-    )
-    (path "/214e5bd1-de3c-4ec2-8553-5b0be1a71a0f/3e20fa31-0809-47c3-be37-022bd242ab1a"
-      (reference "J6") (unit 1) (value "ATARI") (footprint "parts:DIN14")
-    )
-  )
+  )

Commit message: a
Connections:
- net GND: now also J3.1 (Pin_1)
- net FLOPPY_DISKCHANGE: no longer names the net of J4.2 (Pin_2)
- net FLOPPY_DISKCHANGE: no longer J3.1 (Pin_1)
Changed lines of the file:
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@@
+    (stroke (width 0) (type solid) (color 0 0 0 0))
+  )
+  (wire (pts (xy 92.71 50.8) (xy 92.71 52.07))
     (stroke (width 0) (type solid) (color 0 0 0 0))
   )
@@
     (stroke (width 0) (type solid) (color 0 0 0 0))
   )
-  (wire (pts (xy 95.25 44.45) (xy 95.25 52.07))
-    (stroke (width 0) (type solid) (color 0 0 0 0))
-  )
-  (wire (pts (xy 95.25 52.07) (xy 92.71 52.07))
+  (wire (pts (xy 97.79 44.45) (xy 92.71 50.8))
     (stroke (width 0) (type solid) (color 0 0 0 0))
   )
@@
   )
   (wire (pts (xy 115.57 133.35) (xy 120.65 133.35))
-    (stroke (width 0) (type solid) (color 0 0 0 0))
-  )
-  (wire (pts (xy 121.92 44.45) (xy 95.25 44.45))
     (stroke (width 0) (type solid) (color 0 0 0 0))
   )
@@
     (effects (font (size 1.27 1.27)) (justify left bottom))
   )
-  (label "FLOPPY_DISKCHANGE" (at 121.92 44.45 180)
-    (effects (font (size 1.27 1.27)) (justify right bottom))
-  )
   (label "FLOPPY_INDEX" (at 121.92 52.07 180)
     (effects (font (size 1.27 1.27)) (justify right bottom))
@@
     )
     (property "Datasheet" "" (id 3) (at 62.23 43.18 0)
+      (effects (font (size 1.27 1.27)) hide)
+    )
+    (pin "1")
+  )
+  (symbol (lib_id "power:GND") (at 97.79 44.45 0) (unit 1)
+    (in_bom yes) (on_board yes)
+    (property "Reference" "#PWR?" (id 0) (at 97.79 50.8 0)
+      (effects (font (size 1.27 1.27)) hide)
+    )
+    (property "Value" "GND" (id 1) (at 99.06 49.53 0))
+    (property "Footprint" "" (id 2) (at 97.79 44.45 0)
+      (effects (font (size 1.27 1.27)) hide)
+    )
+    (property "Datasheet" "" (id 3) (at 97.79 44.45 0)
       (effects (font (size 1.27 1.27)) hide)
     )
@@
       (reference "#PWR0104") (unit 1) (value "GND") (footprint "")
     )
+    (path "/9bac794a-c4ec-4bd6-8dd4-2f36fa3b4524"
+      (reference "#PWR?") (unit 1) (value "GND") (footprint "")
+    )
     (path "/00000000-0000-0000-0000-00005fc399bb"
